Commit message: update on a lot

File: assets/asset3d/teddy_bear/result/teddy_bear_sim.urdf (robot description, URDF)
Before this commit: robot teddy_bear, 1 links, 0 joints
Links:
- link teddy_bear: mass 0.2000 -> 0.1500; geometry collision mesh filename=mesh/teddy_bear_collision.obj scale=0.154453 0.154453 0.154453; visual mesh filename=mesh/teddy_bear.obj scale=0.154453 0.154453 0.154453
