Commit message: Replace procedural task props with EmbodiedGen V2 assets
Import twelve textured V2 meshes and collision assets, rebuild the existing task and kitchen scenes, refresh the gallery and documentation, and record physical Contract results. Split the kitchen collision proxy at its support levels so counter grasps can be planned; retain honest pot-lift failure evidence.

File: assets/asset3d/foam_cube/result/foam_cube.urdf (robot description, URDF)
Before this commit: robot foam_cube, 1 links, 0 joints
Links:
- link foam_cube: mass 0.035 -> 0.1650; geometry collision mesh filename=mesh/foam_cube_collision.obj scale=1.0 1.0 1.0; visual mesh filename=mesh/foam_cube.obj scale=1.0 1.0 1.0

File: assets/asset3d/foam_cube/result/foam_cube_sim.urdf (robot description, URDF)
Before this commit: robot foam_cube, 1 links, 0 joints
Links:
- link foam_cube: geometry collision mesh filename=mesh/foam_cube_collision.obj scale=0.417327 0.400002 0.401666; visual mesh filename=mesh/foam_cube.obj scale=0.417327 0.400002 0.401666

File: assets/asset3d/handled_cooking_pot/result/handled_cooking_pot.urdf (robot description, URDF)
Before this commit: robot handled_cooking_pot, 1 links, 0 joints
Links:
- link handled_cooking_pot: mass 0.65 -> 2.7500; geometry collision mesh filename=mesh/handled_cooking_pot_collision.obj scale=1.0 1.0 1.0; visual mesh filename=mesh/handled_cooking_pot.obj scale=1.0 1.0 1.0

File: assets/asset3d/handled_cooking_pot/result/handled_cooking_pot_sim.urdf (robot description, URDF)
Before this commit: robot handled_cooking_pot, 1 links, 0 joints
Links:
- link handled_cooking_pot: geometry collision mesh filename=mesh/handled_cooking_pot_collision.obj scale=0.707752 0.492311 0.657391; visual mesh filename=mesh/handled_cooking_pot.obj scale=0.707752 0.492311 0.657391

File: assets/asset3d/juice_bottle/result/juice_bottle.urdf (robot description, URDF)
Before this commit: robot juice_bottle, 1 links, 0 joints
Links:
- link juice_bottle: mass 0.2 -> 0.7500; geometry collision mesh filename=mesh/juice_bottle_collision.obj scale=1.0 1.0 1.0; visual mesh filename=mesh/juice_bottle.obj scale=1.0 1.0 1.0

File: assets/asset3d/juice_bottle/result/juice_bottle_sim.urdf (robot description, URDF)
Before this commit: robot juice_bottle, 1 links, 0 joints
Links:
- link juice_bottle: geometry collision mesh filename=mesh/juice_bottle_collision.obj scale=0.625124 0.765960 0.628041; visual mesh filename=mesh/juice_bottle.obj scale=0.625124 0.765960 0.628041

File: assets/asset3d/paperback_book/result/paperback_book.urdf (robot description, URDF)
Before this commit: robot paperback_book, 1 links, 0 joints
Links:
- link paperback_book: mass 0.25 -> 0.9000; geometry collision mesh filename=mesh/paperback_book_collision.obj scale=1.0 1.0 1.0; visual mesh filename=mesh/paperback_book.obj scale=1.0 1.0 1.0

File: assets/asset3d/paperback_book/result/paperback_book_sim.urdf (robot description, URDF)
Before this commit: robot paperback_book, 1 links, 0 joints
Links:
- link paperback_book: geometry collision mesh filename=mesh/paperback_book_collision.obj scale=0.906093 0.384619 0.887722; visual mesh filename=mesh/paperback_book.obj scale=0.906093 0.384619 0.887722

File: assets/asset3d/plastic_cup/result/plastic_cup.urdf (robot description, URDF)
Before this commit: robot plastic_cup, 1 links, 0 joints
Links:
- link plastic_cup: mass 0.08 -> 0.0250; geometry collision mesh filename=mesh/plastic_cup_collision.obj scale=1.0 1.0 1.0; visual mesh filename=mesh/plastic_cup.obj scale=1.0 1.0 1.0

File: assets/asset3d/plastic_cup/result/plastic_cup_sim.urdf (robot description, URDF)
Before this commit: robot plastic_cup, 1 links, 0 joints
Links:
- link plastic_cup: geometry collision mesh filename=mesh/plastic_cup_collision.obj scale=0.650835 0.678572 0.636108; visual mesh filename=mesh/plastic_cup.obj scale=0.650835 0.678572 0.636108

File: assets/asset3d/rolling_pin/result/rolling_pin.urdf (robot description, URDF)
Before this commit: robot rolling_pin, 1 links, 0 joints
Links:
- link rolling_pin: mass 0.26 -> 0.6000; geometry collision mesh filename=mesh/rolling_pin_collision.obj scale=1.0 1.0 1.0; visual mesh filename=mesh/rolling_pin.obj scale=1.0 1.0 1.0

File: assets/asset3d/rolling_pin/result/rolling_pin_sim.urdf (robot description, URDF)
Before this commit: robot rolling_pin, 1 links, 0 joints
Links:
- link rolling_pin: geometry collision mesh filename=mesh/rolling_pin_collision.obj scale=0.550000 0.550000 0.550000; visual mesh filename=mesh/rolling_pin.obj scale=0.550000 0.550000 0.550000

File: assets/asset3d/shallow_sorting_tray/result/shallow_sorting_tray.urdf (robot description, URDF)
Before this commit: robot shallow_sorting_tray, 1 links, 0 joints
Links:
- link shallow_sorting_tray: mass 0.32 -> 0.3500; geometry collision mesh filename=mesh/shallow_sorting_tray_collision.obj scale=1.0 1.0 1.0; visual mesh filename=mesh/shallow_sorting_tray.obj scale=1.0 1.0 1.0

File: assets/asset3d/shallow_sorting_tray/result/shallow_sorting_tray_sim.urdf (robot description, URDF)
Before this commit: robot shallow_sorting_tray, 1 links, 0 joints
Links:
- link shallow_sorting_tray: geometry collision mesh filename=mesh/shallow_sorting_tray_collision.obj scale=1.167161 0.578956 0.576512; visual mesh filename=mesh/shallow_sorting_tray.obj scale=1.167161 0.578956 0.576512

File: assets/asset3d/small_storage_bin/result/small_storage_bin.urdf (robot description, URDF)
Before this commit: robot small_storage_bin, 1 links, 0 joints
Links:
- link small_storage_bin: mass 0.3 -> 0.7000; geometry collision mesh filename=mesh/small_storage_bin_collision.obj scale=1.0 1.0 1.0; visual mesh filename=mesh/small_storage_bin.obj scale=1.0 1.0 1.0

File: assets/asset3d/small_storage_bin/result/small_storage_bin_sim.urdf (robot description, URDF)
Before this commit: robot small_storage_bin, 1 links, 0 joints
Links:
- link small_storage_bin: geometry collision mesh filename=mesh/small_storage_bin_collision.obj scale=0.712057 0.327276 0.687172; visual mesh filename=mesh/small_storage_bin.obj scale=0.712057 0.327276 0.687172

File: assets/asset3d/snack_carton/result/snack_carton.urdf (robot description, URDF)
Before this commit: robot snack_carton, 1 links, 0 joints
Links:
- link snack_carton: mass 0.18 -> 0.0400; geometry collision mesh filename=mesh/snack_carton_collision.obj scale=1.0 1.0 1.0; visual mesh filename=mesh/snack_carton.obj scale=1.0 1.0 1.0

File: assets/asset3d/snack_carton/result/snack_carton_sim.urdf (robot description, URDF)
Before this commit: robot snack_carton, 1 links, 0 joints
Links:
- link snack_carton: geometry collision mesh filename=mesh/snack_carton_collision.obj scale=0.497357 0.680003 1.058788; visual mesh filename=mesh/snack_carton.obj scale=0.497357 0.680003 1.058788

File: assets/asset3d/soda_can/result/soda_can.urdf (robot description, URDF)
Before this commit: robot soda_can, 1 links, 0 joints
Links:
- link soda_can: mass 0.15 -> 0.0200; geometry collision mesh filename=mesh/soda_can_collision.obj scale=1.0 1.0 1.0; visual mesh filename=mesh/soda_can.obj scale=1.0 1.0 1.0

File: assets/asset3d/soda_can/result/soda_can_sim.urdf (robot description, URDF)
Before this commit: robot soda_can, 1 links, 0 joints
Links:
- link soda_can: geometry collision mesh filename=mesh/soda_can_collision.obj scale=0.845254 0.666670 0.844268; visual mesh filename=mesh/soda_can.obj scale=0.845254 0.666670 0.844268
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