Commit message: SkillNode library: 70 verbs with GT contracts, Isaac Sim verification fixes
- 70 verb SkillNodes (skill_library) with contracts, verifiers and VLM exports
- policy fixes from verification rounds 15-26: pour about the lip, in-air
  upright with staging search, handover grip, bimanual bar grasp, microwave
  cavity withdraw, place finger-slot check, base path keep-out near parks
- left gripper finger collider fix, kitchen layout and prep bowl for pours
- per-step disturbance log in tools/verify_skills.py; docs/PHYSICS_AUDIT.md

Co-Authored-By: Claude Opus 5.5 <noreply@anthropic.com>

File: assets/asset3d/breakfast_bowl/result/breakfast_bowl_sim.urdf (robot description, URDF)
Before this commit: robot breakfast_bowl, 1 links, 0 joints
Links:
- link breakfast_bowl: mass 0.4000 -> 0.2000

File: assets/asset3d/breakfast_mug/result/breakfast_mug_sim.urdf (robot description, URDF)
Before this commit: robot breakfast_mug, 1 links, 0 joints
Links:
- link breakfast_mug: mass 0.3750 -> 0.2500

File: assets/asset3d/breakfast_plate/result/breakfast_plate_sim.urdf (robot description, URDF)
Before this commit: robot breakfast_plate, 1 links, 0 joints
Links:
- link breakfast_plate: mass 0.6000 -> 0.3500

File: assets/asset3d/wide_storage_bin/result/wide_storage_bin_sim.urdf (robot description, URDF)
Before this commit: robot wide_storage_bin, 1 links, 0 joints
Links:
- link wide_storage_bin: mass 1.2000 -> 0.5000
