Commit message: Thin book_red to 4 cm; prepare_assets: per-asset thickness and --patch-usd
The generated red book was 7.0 cm thick. prepare_assets.py gains THICKNESS (resting
height for lay-flat assets, footprint keeps the uniform SPECS scale) and --patch-usd,
which writes the sim URDF's mesh scales, mass and inertia into the existing USD layers
(no EmbodiedGen needed). book_red is now 24 x 16.7 x 4.0 cm, 0.55 kg.

tasks/shelve_books keeps its placements (a --no-reach-check rebuild moved book_green
23 cm and the shelf blocker 19 cm): book_red lowered 15.1 mm in scene.usd/task.json,
then settled, checked and re-annotated.

Co-Authored-By: Claude Opus 5.5 <noreply@anthropic.com>

File: assets/asset3d/book_red/result/book_red_sim.urdf (robot description, URDF)
Before this commit: robot book_red, 1 links, 0 joints
Links:
- link book_red: geometry collision mesh filename=mesh/book_red_collision.obj scale=0.069786 0.040046 0.069786; visual mesh filename=mesh/book_red.obj scale=0.069786 0.040046 0.069786
